Commit message: updated base height

File: model/robot.urdf (robot description, URDF)
Before this commit: robot a1_description, 22 links, 21 joints
Joints:
- joint FL_hip_joint: limit (none) -> effort=20 velocity=52.4
- joint FL_lower_joint: limit (none) -> effort=55 velocity=28.6
- joint FL_upper_joint: limit (none) -> effort=55 velocity=28.6
- joint FR_hip_joint: limit (none) -> effort=20 velocity=52.4
- joint FR_lower_joint: limit (none) -> effort=55 velocity=28.6
- joint FR_upper_joint: limit (none) -> effort=55 velocity=28.6
- joint RL_hip_joint: limit (none) -> effort=20 velocity=52.4
- joint RL_lower_joint: limit (none) -> effort=55 velocity=28.6
- joint RL_upper_joint: limit (none) -> effort=55 velocity=28.6
- joint RR_hip_joint: limit (none) -> effort=20 velocity=52.4
- joint RR_lower_joint: limit (none) -> effort=55 velocity=28.6
- joint RR_upper_joint: limit (none) -> effort=55 velocity=28.6
